File: SCARA_robot/PCB/pcb_controller/pcb_controller.kicad_pcb (KiCad board)
At the start: 2 copper layers, 100 x 100 mm, 60 parts, among them J1 Barrel_Jack_Switch, J10 interface, J11 Conn_01x07_Socket, J15 Conn_01x04_Pin_STEPPER_B, J16 Conn_01x04_Pin_STEPPER_C, J17 Conn_01x02_Pin, J18 Conn_01x04_Pin_STEPPER_C, J19 Conn_01x04_Pin_STEPPER_C, J2 Conn_01x04_Pin_STEPPER_A, J20 Conn_01x04_Pin_STEPPER_C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

Commit message: pcb designed phase 2
Parts:
- moved J7 10.1 mm to (114.3, 116.9), turned to 180 degrees
- moved JP2 6.10 mm to (109.2, 111.3), turned to 90 degrees
- moved J6 2.94 mm to (104.8, 110.0)
- moved J5 0.10 mm to (81.2, 124.6)
Changed lines of the file:
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@@
 	(footprint "Jumper:SolderJumper-3_P1.3mm_Open_RoundedPad1.0x1.5mm"
 		(layer "F.Cu")
-		(at 109 117.4)
+		(at 109.2 111.3 90)
 		(descr "SMD Solder 3-pad Jumper, 1x1.5mm rounded Pads, 0.3mm gap, open")
 		(tags "solder jumper open")
 		(property "Reference" "JP2"
-			(at 0 -1.8 0)
+			(at 0 -1.8 90)
 			(layer "F.SilkS")
 			(effects
@@
 		)
 		(property "Value" "sel_encoderB"
-			(at 0 1.9 0)
+			(at 0 1.9 90)
 			(layer "F.Fab")
 			(effects
@@
 		)
 		(property "Datasheet" ""
-			(at 0 0 0)
+			(at 0 0 90)
 			(unlocked yes)
 			(layer "F.Fab")
@@
 		)
 		(property "Description" "Solder Jumper, 3-pole, open"
-			(at 0 0 0)
+			(at 0 0 90)
 			(unlocked yes)
 			(layer "F.Fab")
@@
 		)
 		(fp_line
-			(start -2.05 0.3)
-			(end -2.05 -0.3)
+			(start -1.4 -1)
+			(end 1.4 -1)
 			(stroke
 				(width 0.12)
@@
 		)
 		(fp_line
-			(start -1.5 1.5)
-			(end -0.9 1.5)
+			(start 2.05 -0.3)
+			(end 2.05 0.3)
 			(stroke
 				(width 0.12)
@@
 		)
 		(fp_line
-			(start -1.4 -1)
-			(end 1.4 -1)
+			(start -2.05 0.3)
+			(end -2.05 -0.3)
 			(stroke
 				(width 0.12)
@@
 		)
 		(fp_line
-			(start -1.2 1.2)
-			(end -1.5 1.5)
+			(start 1.4 1)
+			(end -1.4 1)
 			(stroke
 				(width 0.12)
@@
 		)
 		(fp_line
-			(start 1.4 1)
-			(end -1.4 1)
+			(start -1.2 1.2)
+			(end -1.5 1.5)
 			(stroke
 				(width 0.12)
@@
 		)
 		(fp_line
-			(start 2.05 -0.3)
-			(end 2.05 0.3)
+			(start -1.5 1.5)
+			(end -0.9 1.5)
 			(stroke
 				(width 0.12)
@@
 		)
 		(fp_arc
-			(start -2.05 -0.3)
-			(mid -1.844975 -0.794975)
-			(end -1.35 -1)
+			(start 1.35 -1)
+			(mid 1.844975 -0.794975)
+			(end 2.05 -0.3)
 			(stroke
 				(width 0.12)
@@
 		)
 		(fp_arc
-			(start -1.35 1)
-			(mid -1.844975 0.794975)
-			(end -2.05 0.3)
+			(start -2.05 -0.3)
+			(mid -1.844975 -0.794975)
+			(end -1.35 -1)
 			(stroke
 				(width 0.12)
@@
 		)
 		(fp_arc
-			(start 1.35 -1)
-			(mid 1.844975 -0.794975)
-			(end 2.05 -0.3)
+			(start 2.05 0.3)
+			(mid 1.844975 0.794975)
+			(end 1.35 1)
 			(stroke
 				(width 0.12)
@@
 		)
 		(fp_arc
-			(start 2.05 0.3)
-			(mid 1.844975 0.794975)
-			(end 1.35 1)
+			(start -1.35 1)
+			(mid -1.844975 0.794975)
+			(end -2.05 0.3)
 			(stroke
 				(width 0.12)
@@
 		(fp_line
 			(start -2.3 -1.25)
-			(end -2.3 1.25)
+			(end 2.3 -1.25)
 			(stroke
 				(width 0.05)
@@
 		(fp_line
 			(start -2.3 -1.25)
-			(end 2.3 -1.25)
+			(end -2.3 1.25)
 			(stroke
 				(width 0.05)
@@
 		(fp_line
 			(start 2.3 1.25)
-			(end -2.3 1.25)
+			(end 2.3 -1.25)
 			(stroke
 				(width 0.05)
@@
 		(fp_line
 			(start 2.3 1.25)
-			(end 2.3 -1.25)
+			(end -2.3 1.25)
 			(stroke
 				(width 0.05)
@@
 		)
 		(pad "1" smd custom
-			(at -1.3 0)
+			(at -1.3 0 90)
 			(size 1 0.5)
 			(layers "F.Cu" "F.Mask")
@@
 		)
 		(pad "2" smd rect
-			(at 0 0)
+			(at 0 0 90)
 			(size 1 1.5)
 			(layers "F.Cu" "F.Mask")
@@
 		)
 		(pad "3" smd custom
-			(at 1.3 0)
+			(at 1.3 0 90)
 			(size 1 0.5)
 			(layers "F.Cu" "F.Mask")
@@
 	(footprint "Connector_PinHeader_2.54mm:PinHeader_1x04_P2.54mm_Vertical"
 		(layer "F.Cu")
-		(at 114.3 106.78)
+		(at 114.3 116.9 180)
 		(descr "Through hole straight pin header, 1x04, 2.54mm pitch, single row")
 		(tags "Through hole pin header THT 1x04 2.54mm single row")
@@
 		(attr through_hole)
 		(fp_line
-			(start -1.38 -1.38)
-			(end 0 -1.38)
+			(start 1.38 1.27)
+			(end 1.38 9)
 			(stroke
 				(width 0.12)
@@
 		)
 		(fp_line
-			(start -1.38 0)
-			(end -1.38 -1.38)
+			(start -1.38 9)
+			(end 1.38 9)
 			(stroke
 				(width 0.12)
@@
 		(fp_line
 			(start -1.38 1.27)
-			(end -1.38 9)
+			(end 1.38 1.27)
 			(stroke
 				(width 0.12)
@@
 		(fp_line
 			(start -1.38 1.27)
-			(end 1.38 1.27)
+			(end -1.38 9)
 			(stroke
 				(width 0.12)
@@
 		)
 		(fp_line
-			(start -1.38 9)
-			(end 1.38 9)
+			(start -1.38 0)
+			(end -1.38 -1.38)
 			(stroke
 				(width 0.12)
@@
 		)
 		(fp_line
-			(start 1.38 1.27)
-			(end 1.38 9)
+			(start -1.38 -1.38)
+			(end 0 -1.38)
 			(stroke
 				(width 0.12)
@@
 		)
 		(fp_line
-			(start -1.77 -1.77)
-			(end -1.77 9.39)
+			(start 1.77 9.39)
+			(end 1.77 -1.77)
 			(stroke
 				(width 0.05)
@@
 		)
 		(fp_line
-			(start -1.77 9.39)
-			(end 1.77 9.39)
+			(start 1.77 -1.77)
+			(end -1.77 -1.77)
 			(stroke
 				(width 0.05)
@@
 		)
 		(fp_line
-			(start 1.77 -1.77)
-			(end -1.77 -1.77)
+			(start -1.77 9.39)
+			(end 1.77 9.39)
 			(stroke
 				(width 0.05)
@@
 		)
 		(fp_line
-			(start 1.77 9.39)
-			(end 1.77 -1.77)
+			(start -1.77 -1.77)
+			(end -1.77 9.39)
 			(stroke
 				(width 0.05)
@@
 		)
 		(fp_line
-			(start -1.27 -0.635)
-			(end -0.635 -1.27)
+			(start 1.27 8.89)
+			(end -1.27 8.89)
 			(stroke
 				(width 0.1)
@@
 		)
 		(fp_line
-			(start -1.27 8.89)
-			(end -1.27 -0.635)
+			(start 1.27 -1.27)
+			(end 1.27 8.89)
 			(stroke
 				(width 0.1)
@@
 		)
 		(fp_line
-			(start 1.27 -1.27)
-			(end 1.27 8.89)
+			(start -1.27 8.89)
+			(end -1.27 -0.635)
 			(stroke
 				(width 0.1)
@@
 		)
 		(fp_line
-			(start 1.27 8.89)
-			(end -1.27 8.89)
+			(start -1.27 -0.635)
+			(end -0.635 -1.27)
 			(stroke
 				(width 0.1)
@@
 		)
 		(pad "1" thru_hole rect
-			(at 0 0)
+			(at 0 0 180)
 			(size 1.7 1.7)
 			(drill 1)
@@
 		)
 		(pad "2" thru_hole circle
-			(at 0 2.54)
+			(at 0 2.54 180)
 			(size 1.7 1.7)
 			(drill 1)
@@
 		)
 		(pad "3" thru_hole circle
-			(at 0 5.08)
+			(at 0 5.08 180)
 			(size 1.7 1.7)
 			(drill 1)
@@
 		)
 		(pad "4" thru_hole circle
-			(at 0 7.62)
+			(at 0 7.62 180)
 			(size 1.7 1.7)
 			(drill 1)
@@
 	(footprint "Connector_JST:JST_XH_S7B-XH-A-1_1x07_P2.50mm_Horizontal"
 		(layer "F.Cu")
-		(at 81.3 124.6)
+		(at 81.2 124.6)
 		(descr "JST XH series connector, S7B-XH-A-1 (http://www.jst-mfg.com/product/pdf/eng/eXH.pdf), generated with kicad-footprint-generator")
 		(tags "connector JST XH horizontal")
@@
 	(footprint "Connector_PinHeader_2.54mm:PinHeader_1x03_P2.54mm_Vertical"
 		(layer "F.Cu")
-		(at 105.2 107.11)
+		(at 104.8 110.02)
 		(descr "Through hole straight pin header, 1x03, 2.54mm pitch, single row")
 		(tags "Through hole pin header THT 1x03 2.54mm single row")

Commit message: pcb designed phase 3
Parts:
- J10, J3, J4, J6, J7, J9: moved to B.Cu
- R3: footprint PCM_Resistor_THT_AKL:R_Axial_DIN0204_L3.6mm_D1.6mm_P5.08mm_Horizontal -> PCM_Resistor_THT_AKL:R_Axial_DIN0207_L6.3mm_D2.5mm_P7.62mm_Horizontal
- R4, R5, R6, R7, R8, R9: footprint PCM_Resistor_THT_AKL:R_Axial_DIN0204_L3.6mm_D1.6mm_P5.08mm_Horizontal -> PCM_Resistor_THT_AKL:R_Axial_DIN0207_L6.3mm_D2.5mm_P10.16mm_Horizontal
- moved J7 6.58 mm to (116.2, 110.6)
- moved R6 5.87 mm to (92.5, 73.2)
- moved R8 5.85 mm to (82.6, 73.3)
- moved J3 5.75 mm to (95.1, 110.7)
- moved R7 5.73 mm to (89.3, 73.2)
- moved R9 5.73 mm to (79.5, 73.3)
- moved R5 5.43 mm to (102.7, 73.7)
- moved R4 5.34 mm to (105.8, 73.7)
- moved J10 5.17 mm to (137.3, 110.7)
- moved J9 4.02 mm to (124.6, 110.7)
- moved JP1 3.18 mm to (85.6, 113.1)
- moved JP2 3.11 mm to (106.6, 113.0)
- moved LED1 2.97 mm to (97.5, 36.6)
- moved J4 1.54 mm to (82.4, 110.7), turned to 180 degrees
- moved J6 1.42 mm to (103.5, 110.6), turned to 180 degrees
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Connections:
- JP2 pad 2: /scl_encoderB -> /dirB
Routing:
- net /out_encoderA: track 0.00 -> 22.8 mm
- net /out_encoderC: track 0.00 -> 22.5 mm
- net GNDD_ENA: track 0.00 -> 21.8 mm
- net /dirB: track 0.00 -> 21.7 mm, vias 0 -> 1
- net /out_encoderB: track 0.00 -> 21.5 mm
- net /dirA: track 0.00 -> 21.4 mm, vias 0 -> 1
- net GNDD_ENB: track 0.00 -> 21.1 mm
- net GNDD_ENC: track 0.00 -> 20.8 mm
- net /dirC: track 0.00 -> 19.7 mm, vias 0 -> 1
- net /gpio_encoderA: track 0.00 -> 17.9 mm
- net /gpio_encoderB: track 0.00 -> 17.8 mm
- net /gpio_encoderC: track 0.00 -> 17.5 mm
- net /sda_encoderA: track 0.00 -> 15.1 mm
- net /sda_encoderB: track 0.00 -> 15.1 mm
- net /sda_encoderC: track 0.00 -> 14.9 mm
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
Commit message: pcb finalizada
Parts:
- added ?: , , F.Cu at (148.9, 115.5)
- added ?: , , F.Cu at (149.0, 118.5)
- added ?: , , F.Cu at (148.9, 116.5)
- added ?: , , F.Cu at (149.0, 119.6)
- added ?: , , F.Cu at (148.3, 114.8)
- added ?: , , F.Cu at (148.9, 117.6)
- added mouse-bite-1mm-slot: VAL**, modules:mouse-bite-1mm, F.Cu at (99.9, 132.1)
- added mouse-bite-1mm-slot: VAL**, modules:mouse-bite-1mm, F.Cu at (123.2, 124.0)
- added mouse-bite-1mm-slot: VAL**, modules:mouse-bite-1mm, F.Cu at (123.2, 120.0)
- added mouse-bite-1mm-slot: VAL**, modules:mouse-bite-1mm, F.Cu at (123.1, 132.0)
- added mouse-bite-1mm-slot: VAL**, modules:mouse-bite-1mm, F.Cu at (99.9, 128.1)
- added mouse-bite-1mm-slot: VAL**, modules:mouse-bite-1mm, F.Cu at (126.7, 111.4)
- added mouse-bite-1mm-slot: VAL**, modules:mouse-bite-1mm, F.Cu at (100.0, 109.1)
- added mouse-bite-1mm-slot: VAL**, modules:mouse-bite-1mm, F.Cu at (100.0, 112.0)
- added mouse-bite-1mm-slot: VAL**, modules:mouse-bite-1mm, F.Cu at (123.2, 112.0)
- added mouse-bite-1mm-slot: VAL**, modules:mouse-bite-1mm, F.Cu at (130.7, 111.4)
- added mouse-bite-1mm-slot: VAL**, modules:mouse-bite-1mm, F.Cu at (99.9, 124.0)
- added mouse-bite-1mm-slot: VAL**, modules:mouse-bite-1mm, F.Cu at (99.9, 120.1)
- added mouse-bite-1mm-slot: VAL**, modules:mouse-bite-1mm, F.Cu at (123.2, 109.1)
- added mouse-bite-1mm-slot: VAL**, modules:mouse-bite-1mm, F.Cu at (142.5, 112.2)
- added mouse-bite-1mm-slot: VAL**, modules:mouse-bite-1mm, F.Cu at (123.2, 116.0)
- added mouse-bite-1mm-slot: VAL**, modules:mouse-bite-1mm, F.Cu at (100.0, 116.0)
- added mouse-bite-1mm-slot: VAL**, modules:mouse-bite-1mm, F.Cu at (123.1, 128.1)
- added mouse-bite-1mm-slot: VAL**, modules:mouse-bite-1mm, F.Cu at (146.0, 113.8)
- added mouse-bite-5mm-slot: VAL**, modules:mouse-bite-5mm-slot, F.Cu at (84.9, 105.1)
- added mouse-bite-5mm-slot: VAL**, modules:mouse-bite-5mm-slot, F.Cu at (94.9, 105.1)
- added mouse-bite-5mm-slot: VAL**, modules:mouse-bite-5mm-slot, F.Cu at (124.8, 105.2)
- added mouse-bite-5mm-slot: VAL**, modules:mouse-bite-5mm-slot, F.Cu at (133.9, 108.0)
- added mouse-bite-5mm-slot: VAL**, modules:mouse-bite-5mm-slot, F.Cu at (114.8, 105.2)
- added mouse-bite-5mm-slot: VAL**, modules:mouse-bite-5mm-slot, F.Cu at (151.4, 126.4)
- added mouse-bite-5mm-slot: VAL**, modules:mouse-bite-5mm-slot, F.Cu at (104.8, 105.1)
- moved J9 22.9 mm to (146.6, 117.1), turned to 90 degrees
- moved J10 21.2 mm to (146.6, 129.8), turned to 90 degrees
- moved JP3 18.0 mm to (144.2, 120.2), turned to 0 degrees
- moved J11 12.6 mm to (132.7, 116.0), turned to -90 degrees
- moved J6 1.62 mm to (105.0, 110.0)
- moved JP2 1.62 mm to (108.1, 112.5)
- moved J7 1.62 mm to (117.7, 110.0)
- moved J8 1.62 mm to (103.9, 124.0)
- moved J4 0.74 mm to (81.9, 110.2)
- moved J3 0.74 mm to (94.6, 110.2)
- moved J5 0.74 mm to (80.7, 124.1)
- moved JP1 0.74 mm to (85.1, 112.6)

Commit message: pcb finalizada, todo revisar
Parts:
- removed the mouse-bite-1mm-slot at (123.2, 124.0)
- removed the mouse-bite-1mm-slot at (123.2, 120.0)
- removed the mouse-bite-1mm-slot at (123.1, 132.0)
- removed the mouse-bite-1mm-slot at (123.2, 112.0)
- removed the mouse-bite-1mm-slot at (123.2, 109.1)
- removed the mouse-bite-1mm-slot at (123.2, 116.0)
- removed the mouse-bite-1mm-slot at (123.1, 128.1)
- added Adrián Silva Palafox: LOGO, modules:LOGOFOURIEREMBEDS, F.Cu at (89.7, 60.9)
- added mouse-bite-1mm-slot: VAL**, modules:mouse-bite-1mm, F.Cu at (123.2, 109.1)
- added mouse-bite-1mm-slot: VAL**, modules:mouse-bite-1mm, F.Cu at (123.2, 130.1)
- added mouse-bite-1mm-slot: VAL**, modules:mouse-bite-1mm, F.Cu at (123.2, 124.1)
- added mouse-bite-1mm-slot: VAL**, modules:mouse-bite-1mm, F.Cu at (123.2, 115.1)
- added mouse-bite-1mm-slot: VAL**, modules:mouse-bite-1mm, F.Cu at (100.0, 133.1)
- added mouse-bite-1mm-slot: VAL**, modules:mouse-bite-1mm, F.Cu at (123.2, 127.1)
- added mouse-bite-1mm-slot: VAL**, modules:mouse-bite-1mm, F.Cu at (123.2, 118.1)
- added mouse-bite-1mm-slot: VAL**, modules:mouse-bite-1mm, F.Cu at (123.2, 121.1)
- added mouse-bite-1mm-slot: VAL**, modules:mouse-bite-1mm, F.Cu at (123.2, 133.1)
- added mouse-bite-1mm-slot: VAL**, modules:mouse-bite-1mm, F.Cu at (100.0, 130.1)
- added mouse-bite-1mm-slot: VAL**, modules:mouse-bite-1mm, F.Cu at (123.2, 112.0)
- moved mouse-bite-1mm-slot 4.95 mm to (100.0, 127.1)
- moved mouse-bite-1mm-slot 3.98 mm to (100.0, 124.1)
- moved mouse-bite-1mm-slot 2.98 mm to (100.0, 121.1)
- moved mouse-bite-1mm-slot 2.00 mm to (100.0, 118.1)
- moved mouse-bite-1mm-slot 0.95 mm to (100.0, 115.1)
- moved mouse-bite-1mm-slot 0.41 mm to (130.6, 111.0)
Routing:
- net +3.3V: track 260.9 -> 264.2 mm
- net /out_encoderC: track 22.5 -> 20.3 mm
- net +12V: track 270.1 -> 268.5 mm
- net +5V: track 57.8 -> 56.6 mm
- net /baseM_rst: track 62.2 -> 61.2 mm
- net /link2_rst: track 61.9 -> 61.3 mm
Other:
- outline, holes or cut-outs redrawn
- board text added: "12V"
- board text added: "3.3v out gnd scl sda gpio"
- board text added: "A2|A1|B1|B2"
- board text added: "Encoders AS5600 interfaces 4 | 3 | 2 | 1 sda | scl | gnd | 3.3v"
- board text added: "M0 | M1 | M2"
- board text added: "Scara robot controller board ---------------- Designed by: Adrián Silva Palafox"
