File: SCARA_robot/PCB/pcb_controller/pcb_controller.kicad_pcb (KiCad board)
At the start: 2 copper layers, 100 x 100 mm, 96 parts, among them J1 Barrel_Jack_Switch, J10 interface, J11 Conn_01x07_Socket, J15 Conn_01x04_Pin_STEPPER_B, J16 Conn_01x04_Pin_STEPPER_C, J17 Conn_01x02_Pin, J18 Conn_01x04_Pin_STEPPER_C, J19 Conn_01x04_Pin_STEPPER_C, J2 Conn_01x04_Pin_STEPPER_A, J20 Conn_01x04_Pin_STEPPER_C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

Commit message: rediseño de PCB
Parts:
- removed ? (x6): , 
- removed mouse-bite-1mm-slot (x22): VAL**, modules:mouse-bite-1mm
- removed mouse-bite-5mm-slot (x7): VAL**, modules:mouse-bite-5mm-slot
- D2, J10, J3, J4, J6, J7, J9, R4, R5, R6, R7, R8, R9, U1: moved to F.Cu
- moved J10 104.4 mm to (70.7, 58.2), turned to 0 degrees
- moved J9 102.3 mm to (70.7, 48.5), turned to 0 degrees
- moved J11 99.4 mm to (40.7, 78.2), turned to 0 degrees
- moved JP3 92.6 mm to (62.0, 77.5)
- moved Adrián Silva Palafox 87.0 mm to (147.0, 126.4)
- moved J8 86.7 mm to (40.7, 64.7)
- moved J5 83.2 mm to (40.7, 51.1)
- moved J7 73.2 mm to (66.1, 58.2), turned to 0 degrees
- moved J6 72.8 mm to (66.1, 48.5), turned to 0 degrees
- moved J4 65.0 mm to (61.5, 48.5), turned to 0 degrees
- moved J3 61.6 mm to (61.5, 58.2), turned to 0 degrees
- moved JP2 60.2 mm to (62.0, 73.7), turned to 0 degrees
- moved R5 58.0 mm to (131.2, 124.2), turned to 180 degrees
- moved R6 57.2 mm to (118.5, 124.2), turned to 180 degrees
- moved R4 54.9 mm to (133.7, 121.0), turned to 180 degrees
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Connections:
- U2 pad 11: /sda_master -> /scl_master
- U2 pad 14: /scl_master -> /sda_master
Routing:
- net +12V: track 268.5 -> 209.6 mm, vias 0 -> 4
- net +3.3V: track 264.3 -> 318.6 mm, vias 2 -> 0
- net +5V: track 56.6 -> 102.2 mm
- net /rst_master: track 29.9 -> 57.9 mm
- net /out_encoderA: track 22.5 -> 0.00 mm
- net GNDD_ENA: track 21.7 -> 0.00 mm
- net /dirB: track 21.6 -> 0.00 mm, vias 1 -> 0
- net /dirA: track 21.3 -> 0.00 mm, vias 1 -> 0
- net /out_encoderB: track 21.2 -> 0.00 mm
- net GNDD_ENB: track 20.9 -> 0.00 mm
- net GNDD_ENC: track 20.5 -> 0.00 mm
- net /out_encoderC: track 20.3 -> 0.00 mm
- net /sda_master: track 13.3 -> 32.9 mm
- net /dirC: track 19.5 -> 0.00 mm, vias 1 -> 0
- net /scl_master: track 21.6 -> 40.0 mm
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Other:
- outline, holes or cut-outs redrawn
- board text removed: "3.3v out gnd scl sda gpio"

Commit message: Encoders' shield added
Parts:
- removed J10, J7: interface, Connector_PinHeader_2.54mm:PinHeader_1x04_P2.54mm_Vertical
- removed J11, J8: Conn_01x07_Socket, Connector_JST:JST_XH_S7B-XH-A-1_1x07_P2.50mm_Horizontal
- removed J6, J9: power, Connector_PinHeader_2.54mm:PinHeader_1x03_P2.54mm_Vertical
- removed JP2: sel_encoderB, Jumper:SolderJumper-3_P1.3mm_Open_RoundedPad1.0x1.5mm
- removed JP3: sel_encoderC, Jumper:SolderJumper-3_P1.3mm_Open_RoundedPad1.0x1.5mm
- moved J4 87.3 mm to (23.8, 127.2), turned to 180 degrees
- moved J5 84.4 mm to (22.3, 133.5)
- moved J3 73.5 mm to (36.3, 127.2), turned to 180 degrees
- moved JP1 63.2 mm to (28.5, 123.4), turned to -90 degrees
- moved A1 60.5 mm to (106.3, 47.8)
- moved Adrián Silva Palafox 60.5 mm to (88.9, 109.3)
- moved C1 60.5 mm to (110.6, 29.1)
- moved J15 60.5 mm to (114.7, 64.1)
- moved J17 60.5 mm to (84.4, 22.6)
- moved J19 60.5 mm to (56.1, 113.7)
- moved J2 60.5 mm to (115.2, 37.7)
- moved J20 60.5 mm to (42.5, 113.6)
- moved JP4 60.5 mm to (99.5, 42.7)
- moved JP5 60.5 mm to (99.1, 69.5)
- moved R3 60.5 mm to (33.4, 40.4)
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Routing:
- net /dirA: track 0.00 -> 39.0 mm
- net +3.3V_ENA: track 0.00 -> 19.3 mm
- net GNDD_ENA: track 0.00 -> 14.7 mm
- net /scl_encoderA: track 0.00 -> 14.3 mm
- net /out_encoderA: track 0.00 -> 11.7 mm
- net /sda_encoderA: track 0.00 -> 10.7 mm
- net /gpio_encoderA: track 0.00 -> 6.63 mm
- added copper zone on F.Cu, net GNDD_ENA
Other:
- board size 100 x 100 mm -> 100 x 119.4 mm
