File: SCARA_robot/PCB/pcb_controller/pcb_controller.kicad_sch (KiCad schematic)
At the start: 60 parts, among them J1 Barrel_Jack_Switch, J10 interface, J11 Conn_01x07_Socket, J15 Conn_01x04_Pin_STEPPER_B, J16 Conn_01x04_Pin_STEPPER_C, J17 Conn_01x02_Pin, J18 Conn_01x04_Pin_STEPPER_C, J19 Conn_01x04_Pin_STEPPER_C, J2 Conn_01x04_Pin_STEPPER_A, J20 Conn_01x04_Pin_STEPPER_C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

Commit message: pcb designed phase 3
Parts:
- R3: footprint PCM_Resistor_THT_AKL:R_Axial_DIN0204_L3.6mm_D1.6mm_P5.08mm_Horizontal -> PCM_Resistor_THT_AKL:R_Axial_DIN0207_L6.3mm_D2.5mm_P7.62mm_Horizontal
- R4, R5, R6, R7, R8, R9: footprint PCM_Resistor_THT_AKL:R_Axial_DIN0204_L3.6mm_D1.6mm_P5.08mm_Horizontal -> PCM_Resistor_THT_AKL:R_Axial_DIN0207_L6.3mm_D2.5mm_P10.16mm_Horizontal
Connections:
- net dirB: now also JP2.2 (C)
- net scl_encoderB: no longer JP2.2 (C)
Changed lines of the file:
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@@
 	)
 	(junction
-		(at 33.02 140.97)
-		(diameter 0)
-		(color 0 0 0 0)
-	)
-	(junction
 		(at 68.58 67.31)
 		(diameter 0)
@@
 	)
 	(junction
+		(at 33.02 138.43)
+		(diameter 0)
+		(color 0 0 0 0)
+	)
+	(junction
 		(at 193.04 26.67)
 		(diameter 0)
@@
 	(wire
 		(pts
-			(xy 33.02 140.97) (xy 33.02 147.32)
-		)
-		(stroke
-			(width 0)
-			(type default)
-		)
-	)
-	(wire
-		(pts
 			(xy 31.75 167.64) (xy 58.42 167.64)
 		)
@@
 	(wire
 		(pts
+			(xy 33.02 138.43) (xy 59.69 138.43)
+		)
+		(stroke
+			(width 0)
+			(type default)
+		)
+	)
+	(wire
+		(pts
 			(xy 273.05 91.44) (xy 265.43 91.44)
 		)
@@
 	(wire
 		(pts
-			(xy 33.02 140.97) (xy 59.69 140.97)
-		)
-		(stroke
-			(width 0)
-			(type default)
-		)
-	)
-	(wire
-		(pts
 			(xy 134.62 45.72) (xy 135.89 45.72)
 		)
@@
 	(wire
 		(pts
-			(xy 31.75 140.97) (xy 33.02 140.97)
+			(xy 31.75 140.97) (xy 59.69 140.97)
 		)
 		(stroke
@@
 		)
 	)
+	(wire
+		(pts
+			(xy 33.02 138.43) (xy 33.02 147.32)
+		)
+		(stroke
+			(width 0)
+			(type default)
+		)
+	)
 	(polyline
 		(pts
@@
 	(wire
 		(pts
-			(xy 31.75 138.43) (xy 59.69 138.43)
+			(xy 31.75 138.43) (xy 33.02 138.43)
 		)
 		(stroke
@@
 			)
 		)
-		(property "Footprint" "PCM_Resistor_THT_AKL:R_Axial_DIN0204_L3.6mm_D1.6mm_P5.08mm_Horizontal"
+		(property "Footprint" "PCM_Resistor_THT_AKL:R_Axial_DIN0207_L6.3mm_D2.5mm_P10.16mm_Horizontal"
 			(at 176.53 33.02 0)
 			(effects
@@
 			)
 		)
-		(property "Footprint" "PCM_Resistor_THT_AKL:R_Axial_DIN0204_L3.6mm_D1.6mm_P5.08mm_Horizontal"
+		(property "Footprint" "PCM_Resistor_THT_AKL:R_Axial_DIN0207_L6.3mm_D2.5mm_P10.16mm_Horizontal"
 			(at 185.42 33.02 0)
 			(effects
@@
 			)
 		)
-		(property "Footprint" "PCM_Resistor_THT_AKL:R_Axial_DIN0204_L3.6mm_D1.6mm_P5.08mm_Horizontal"
+		(property "Footprint" "PCM_Resistor_THT_AKL:R_Axial_DIN0207_L6.3mm_D2.5mm_P10.16mm_Horizontal"
 			(at 208.28 33.02 0)
 			(effects
@@
 			)
 		)
-		(property "Footprint" "PCM_Resistor_THT_AKL:R_Axial_DIN0204_L3.6mm_D1.6mm_P5.08mm_Horizontal"
+		(property "Footprint" "PCM_Resistor_THT_AKL:R_Axial_DIN0207_L6.3mm_D2.5mm_P10.16mm_Horizontal"
 			(at 193.04 33.02 0)
 			(effects
@@
 			)
 		)
-		(property "Footprint" "PCM_Resistor_THT_AKL:R_Axial_DIN0204_L3.6mm_D1.6mm_P5.08mm_Horizontal"
+		(property "Footprint" "PCM_Resistor_THT_AKL:R_Axial_DIN0207_L6.3mm_D2.5mm_P7.62mm_Horizontal"
 			(at 93.98 30.48 0)
 			(effects
@@
 			)
 		)
-		(property "Footprint" "PCM_Resistor_THT_AKL:R_Axial_DIN0204_L3.6mm_D1.6mm_P5.08mm_Horizontal"
+		(property "Footprint" "PCM_Resistor_THT_AKL:R_Axial_DIN0207_L6.3mm_D2.5mm_P10.16mm_Horizontal"
 			(at 200.66 33.02 0)
 			(effects
@@
 			)
 		)
-		(property "Footprint" "PCM_Resistor_THT_AKL:R_Axial_DIN0204_L3.6mm_D1.6mm_P5.08mm_Horizontal"
+		(property "Footprint" "PCM_Resistor_THT_AKL:R_Axial_DIN0207_L6.3mm_D2.5mm_P10.16mm_Horizontal"
 			(at 168.91 33.02 0)
 			(effects

Commit message: rediseño de PCB
Connections:
- net scl_master: now also U2.11 (D21); no longer U2.14 (D22)
- net sda_master: now also U2.14 (D22); no longer U2.11 (D21)
Changed lines of the file:
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@@
-		)
-	)
-	(label "scl_master"
-		(at 175.26 124.46 0)
-		(effects
-			(font
-				(size 1.27 1.27)
-			)
-			(justify left bottom)
 		)
 	)
@@
 		)
 	)
-	(label "sda_master"
-		(at 142.24 147.32 180)
-		(effects
-			(font
-				(size 1.27 1.27)
-			)
-			(justify right bottom)
-		)
-	)
 	(label "sda_enB"
 		(at 85.09 140.97 0)
@@
 			)
 			(justify right bottom)
+		)
+	)
+	(label "sda_master"
+		(at 175.26 124.46 0)
+		(effects
+			(font
+				(size 1.27 1.27)
+			)
+			(justify left bottom)
 		)
 	)
@@
 		)
 	)
+	(label "scl_master"
+		(at 142.24 147.32 180)
+		(effects
+			(font
+				(size 1.27 1.27)
+			)
+			(justify right bottom)
+		)
+	)
