Commit message: my_robot with urdf examples

File: drawer_robot/my_robot.urdf (robot description, URDF)
Before this commit: robot my_robot, 1 links, 0 joints
Links:
- added link shoulder_link; visual cylinder length=0.3 radius=0.1
- link base_link: geometry visual box size=0.6 0.4 0.2
Joints:
- added joint base_shoulder_joint: type revolute, parent base_link, child shoulder_link, origin xyz=0 0 0.2 rpy=0 0 0, axis 0 0 1, limit lower=-3.14 upper=3.14 effort=100 velocity=100
