Commit message: my_car_description pkg

File: drawer_robot/my_car.urdf.xacro (robot description, xacro)
@@ -1,10 +1,17 @@
 <?xml version="1.0"?>
 <!--
-    Archivo URDF para definir un robot móvil simple llamado "my_car".
+    Archivo Xacro para definir un robot móvil simple llamado "my_car".
     Este robot tiene un cuerpo principal (base_link), dos ruedas delanteras (con articulaciones continuas)
     y una rueda trasera tipo caster (articulación fija). También incluye un enlace virtual para la base.
     Puede ser utilizado en simuladores como Gazebo o visualizado en RViz.
 -->
-<robot name="my_car">
+<robot name="my_car" xmlns:xacro="http://www.ros.org/wiki/xacro">
+    <!-- Propiedades reutilizables -->
+    <xacro:property name="base_length" value="0.6"/> <!-- Longitud de la base -->
+    <xacro:property name="base_width" value="0.4"/> <!-- Ancho de la base -->
+    <xacro:property name="base_height" value="0.2"/> <!-- Altura de la base -->
+    <xacro:property name="wheel_radius" value="0.1"/> <!-- Radio de las ruedas -->
+    <xacro:property name="wheel_length" value="0.05"/> <!-- Ancho de las ruedas -->
+    <xacro:property name="caster_radius" value="0.05"/> <!-- Radio de la rueda trasera tipo caster -->
     <!-- Definición de materiales -->
     <material name="green">
@@ -14,38 +21,34 @@
         <color rgba="0.5 0.5 0.5 1"/> <!-- Color gris -->
     </material>
+    <!-- Macro para la definición de una rueda-->
+    <xacro:macro name="wheel_link" params="prefix">
+        <link name="wheel_front_${prefix}">
+            <visual>
+                <geometry>
+                    <cylinder radius="${wheel_radius}" length="${wheel_length}"/> <!-- Cilindro con dimensiones definidas por propiedades -->
+                </geometry>
+                <origin xyz="0 0 0" rpy="${pi / 2.0} 0 0"/> <!-- Orientación para que sea perpendicular al suelo -->
+                <material name="grey"/> <!-- Material gris -->
+            </visual>
+        </link>
+    </xacro:macro>
     <!-- Definición del enlace base (base_link) -->
     <link name="base_link">
         <visual>
             <geometry>
-                <box size="0.6 0.4 0.2"/> <!-- Caja con dimensiones 0.6 x 0.4 x 0.2 -->
+                <box size="${base_length} ${base_width} ${base_height}"/> <!-- Caja con dimensiones definidas por propiedades -->
             </geometry>
-            <origin xyz="0 0 0.1" rpy="0 0 0"/> <!-- Posición del enlace en el marco de coordenadas -->
+            <origin xyz="0 0 ${base_height / 2.0}" rpy="0 0 0"/> <!-- Posición del enlace en el marco de coordenadas -->
             <material name="green"/> <!-- Material verde -->
         </visual>
     </link>
     <!-- Definición de las ruedas delanteras -->
-    <link name="wheel_front_left">
-        <visual>
-            <geometry>
-                <cylinder radius="0.1" length="0.05"/> <!-- Cilindro con radio 0.1 y longitud 0.05 -->
-            </geometry>
-            <origin xyz="0 0 0" rpy="1.57 0 0"/> <!-- Orientación para que sea perpendicular al suelo -->
-            <material name="grey"/> <!-- Material gris -->
-        </visual>
-    </link>
-    <link name="wheel_front_right">
-        <visual>
-            <geometry>
-                <cylinder radius="0.1" length="0.05"/> <!-- Cilindro con radio 0.1 y longitud 0.05 -->
-            </geometry>
-            <origin xyz="0 0 0" rpy="1.57 0 0"/> <!-- Orientación para que sea perpendicular al suelo -->
-            <material name="grey"/> <!-- Material gris -->
-        </visual>
-    </link>
+    <xacro:wheel_link prefix="left"/> <!-- Rueda delantera izquierda -->
+    <xacro:wheel_link prefix="right"/> <!-- Rueda delantera derecha -->
     <!-- Definición de la rueda trasera tipo caster -->
     <link name="caster_wheel">
         <visual>
             <geometry>
-                <sphere radius="0.05"/> <!-- Esfera con radio 0.05 -->
+                <sphere radius="${caster_radius}"/> <!-- Esfera con radio definido por propiedad -->
             </geometry>
             <origin xyz="0 0 0" rpy="0 0 0"/> <!-- Posición en el marco de coordenadas -->
@@ -60,5 +63,5 @@
         <parent link="base_link"/> <!-- Enlace padre -->
         <child link="wheel_front_left"/> <!-- Enlace hijo -->
-        <origin xyz="-0.15 -0.225 0" rpy="0 0 0"/> <!-- Posición de la articulación -->
+        <origin xyz="-${base_length / 4.0} -${base_width / 2.0 - wheel_radius} 0" rpy="0 0 0"/> <!-- Posición de la articulación -->
         <axis xyz="0 1 0"/> <!-- Eje de rotación (Y) -->
     </joint>
@@ -67,5 +70,5 @@
         <parent link="base_link"/> <!-- Enlace padre -->
         <child link="wheel_front_right"/> <!-- Enlace hijo -->
-        <origin xyz="-0.15 0.225 0" rpy="0 0 0"/> <!-- Posición de la articulación -->
+        <origin xyz="-${base_length / 4.0} ${base_width / 2.0 - wheel_radius} 0" rpy="0 0 0"/> <!-- Posición de la articulación -->
         <axis xyz="0 1 0"/> <!-- Eje de rotación (Y) -->
     </joint>
@@ -74,5 +77,5 @@
         <parent link="base_link"/> <!-- Enlace padre -->
         <child link="caster_wheel"/> <!-- Enlace hijo -->
-        <origin xyz="0.2 0 -0.05" rpy="0 0 0"/> <!-- Posición de la articulación -->
+        <origin xyz="${base_length / 3.0} 0 -${caster_radius}" rpy="0 0 0"/> <!-- Posición de la articulación -->
     </joint>
     <!-- Articulación fija entre base_footprint y base_link -->
@@ -80,5 +83,5 @@
         <parent link="base_footprint"/> <!-- Enlace padre -->
         <child link="base_link"/> <!-- Enlace hijo -->
-        <origin xyz="0 0 0.1" rpy="0 0 0"/> <!-- Posición de la articulación -->
+        <origin xyz="0 0 ${base_height / 2.0}" rpy="0 0 0"/> <!-- Posición de la articulación -->
     </joint>
 </robot>

File: drawer_robot/my_robot.urdf.xacro (robot description, xacro)
@@ -5,5 +5,5 @@
     Puede ser utilizado en simuladores como Gazebo o visualizado en RViz.
 -->
-<robot name="my_robot">
+<robot name="my_robot" xmlns:xacro="http://www.ros.org/wiki/xacro">
     <!-- Definición de materiales -->
     <material name="green">
