Commit message: my_car_description pkg

File: drawer_robot/my_car_ws/src/my_car_description/urdf/mobile_base.xacro (robot description, xacro)
@@ -2,9 +2,9 @@
 <robot xmlns:xacro="http://www.ros.org/wiki/xacro">
     <!-- Propiedades reutilizables -->
-    <xacro:property name="base_length" value="0.6"/> <!-- Longitud de la base -->
-    <xacro:property name="base_width" value="0.4"/> <!-- Ancho de la base -->
-    <xacro:property name="base_height" value="0.2"/> <!-- Altura de la base -->
-    <xacro:property name="wheel_radius" value="0.1"/> <!-- Radio de las ruedas -->
-    <xacro:property name="wheel_length" value="0.05"/> <!-- Ancho de las ruedas -->
+    <xacro:property name="base_length" value="0.6"/>    <!-- Longitud de la base -->
+    <xacro:property name="base_width" value="0.4"/>     <!-- Ancho de la base -->
+    <xacro:property name="base_height" value="0.2"/>    <!-- Altura de la base -->
+    <xacro:property name="wheel_radius" value="0.1"/>   <!-- Radio de las ruedas -->
+    <xacro:property name="wheel_length" value="0.05"/>  <!-- Ancho de las ruedas -->
     <xacro:property name="caster_radius" value="0.05"/> <!-- Radio de la rueda trasera tipo caster -->
     <!-- Macro para la definición de una rueda-->
